Commit message: add mars_lite xacro mu1 mu2 & turtlebot3 gmapping lidar range up & added map.yaml

File: master_robot/mars_ws/src/mars_lite_description/urdf/mars_lite_with_gripper.urdf.xacro (robot description, xacro)
@@ -173,6 +173,6 @@
     <inertial>
       <origin xyz="0 0 0" rpy="0 0 0"/>
-      <mass value="5.0" />
-      <xacro:box_inertia m="5.0" x="${tm_cntrl_box_length}" y="${tm_cntrl_box_width}" z="${tm_cntrl_box_height}" />
+      <mass value="0.01" />
+      <xacro:box_inertia m="0.01" x="${tm_cntrl_box_length}" y="${tm_cntrl_box_width}" z="${tm_cntrl_box_height}" />
     </inertial>
   </link>

Commit message: static_individual_exp comparison done

File: master_robot/mars_ws/src/mars_lite_description/urdf/mars_lite_with_gripper.urdf.xacro (robot description, xacro)
@@ -150,6 +150,6 @@
       <inertial>
         <origin xyz="0 0 0" rpy="0 0 0" />
-        <mass value="2.0" />
-        <xacro:cylinder_inertia m="10" r="${wheel_radius}" h="0.03" />
+        <mass value="20.0" />
+        <xacro:cylinder_inertia m="20" r="${wheel_radius}" h="0.03" />
       </inertial>
     </link>
